File: Relay.sch (KiCad schematic (older format))
At the start: 0 parts

Commit message: Rough schematic created for relay circuit
Parts:
- added D?: LED, symbol LED
- added D?: DIODE, symbol DIODE
- added K?: RELAY_SPDT, symbol RELAY_SPDT
- added Q?: NPN, symbol NPN
- added R? (x6): R, symbol R
- added U?: PHTRANS, symbol PHTRANS
Connections:
- net labels added: +12V, COM, GND, NC, NO
- net labels removed: Relay+, Relay-
- wire segments 0 -> 29
Changed lines of the file:
@@
 $Descr A4 11693 8268
 encoding utf-8
-Sheet 4 8
+Sheet 3 8
 Title ""
 Date ""
@@
 Comment4 ""
 $EndDescr
-Text HLabel 2400 2300 0    60   Input ~ 0
+Text HLabel 2000 2800 0    60   Input ~ 0
 DIN+
-Text HLabel 2400 2500 0    60   Output ~ 0
+Text HLabel 2000 3150 0    60   Output ~ 0
 DIN-
-Text HLabel 8800 2300 0    60   Input ~ 0
-Relay+
-Text HLabel 8800 2500 0    60   Output ~ 0
-Relay-
+Text HLabel 8300 2250 2    60   BiDi ~ 0
+NC
+Text HLabel 8300 2450 2    60   BiDi ~ 0
+NO
+$Comp
+L PHTRANS U?
+U 1 1 52F15ED8
+P 3850 3000
+F 0 "U?" H 3800 3350 70  0000 C CNN
+F 1 "PHTRANS" H 3800 2650 70  0000 C CNN
+F 2 "" H 3850 3000 60  0000 C CNN
+F 3 "" H 3850 3000 60  0000 C CNN
+	1    3850 3000
+	1    0    0    -1
+$EndComp
+$Comp
+L R R?
+U 1 1 52F15EEC
+P 5650 3200
+F 0 "R?" V 5730 3200 40  0000 C CNN
+F 1 "R" V 5657 3201 40  0000 C CNN
+F 2 "" V 5580 3200 30  0000 C CNN
+F 3 "" H 5650 3200 30  0000 C CNN
+	1    5650 3200
+	0    -1   -1   0
+$EndComp
+$Comp
+L NPN Q?
+U 1 1 52F15F00
+P 6800 3600
+F 0 "Q?" H 6800 3450 50  0000 R CNN
+F 1 "NPN" H 6800 3750 50  0000 R CNN
+F 2 "" H 6800 3600 60  0000 C CNN
+F 3 "" H 6800 3600 60  0000 C CNN
+	1    6800 3600
+	1    0    0    -1
+$EndComp
+$Comp
+L LED D?
+U 1 1 52F15F14
+P 5100 3600
+F 0 "D?" H 5100 3700 50  0000 C CNN
+F 1 "LED" H 5100 3500 50  0000 C CNN
+F 2 "" H 5100 3600 60  0000 C CNN
+F 3 "" H 5100 3600 60  0000 C CNN
+	1    5100 3600
+	0    1    1    0
+$EndComp
+$Comp
+L RELAY_SPDT K?
+U 1 1 52F16219
+P 7450 2300
+F 0 "K?" H 7450 2550 70  0000 C CNN
+F 1 "RELAY_SPDT" H 7450 1750 70  0000 C CNN
+F 2 "" H 7450 2300 60  0000 C CNN
+F 3 "" H 7450 2300 60  0000 C CNN
+	1    7450 2300
+	1    0    0    -1
+$EndComp
+Text HLabel 8300 1850 2    60   BiDi ~ 0
+COM
+$Comp
+L R R?
+U 1 1 52F162BB
+P 6900 4250
+F 0 "R?" V 6980 4250 40  0000 C CNN
+F 1 "R" V 6907 4251 40  0000 C CNN
+F 2 "" V 6830 4250 30  0000 C CNN
+F 3 "" H 6900 4250 30  0000 C CNN
+	1    6900 4250
+	-1   0    0    1
+$EndComp
+$Comp
+L GND #PWR?
+U 1 1 52F162E0
+P 6900 4800
+F 0 "#PWR?" H 6900 4800 30  0001 C CNN
+F 1 "GND" H 6900 4730 30  0001 C CNN
+F 2 "" H 6900 4800 60  0000 C CNN
+F 3 "" H 6900 4800 60  0000 C CNN
+	1    6900 4800
+	1    0    0    -1
+$EndComp
+$Comp
+L R R?
+U 1 1 52F162FC
+P 5100 4250
+F 0 "R?" V 5180 4250 40  0000 C CNN
+F 1 "R" V 5107 4251 40  0000 C CNN
+F 2 "" V 5030 4250 30  0000 C CNN
+F 3 "" H 5100 4250 30  0000 C CNN
+	1    5100 4250
+	-1   0    0    1
+$EndComp
+$Comp
+L +12V #PWR?
+U 1 1 52F16338
+P 5900 1500
+F 0 "#PWR?" H 5900 1450 20  0001 C CNN
+F 1 "+12V" H 5900 1600 30  0000 C CNN
+F 2 "" H 5900 1500 60  0000 C CNN
+F 3 "" H 5900 1500 60  0000 C CNN
+	1    5900 1500
+	1    0    0    -1
+$EndComp
+$Comp
+L R R?
+U 1 1 52F16354
+P 5900 1950
+F 0 "R?" V 5980 1950 40  0000 C CNN
+F 1 "R" V 5907 1951 40  0000 C CNN
+F 2 "" V 5830 1950 30  0000 C CNN
+F 3 "" H 5900 1950 30  0000 C CNN
+	1    5900 1950
+	-1   0    0    1
+$EndComp
+$Comp
+L R R?
+U 1 1 52F16372
+P 4950 2800
+F 0 "R?" V 5030 2800 40  0000 C CNN
+F 1 "R" V 4957 2801 40  0000 C CNN
+F 2 "" V 4880 2800 30  0000 C CNN
+F 3 "" H 4950 2800 30  0000 C CNN
+	1    4950 2800
+	0    1    1    0
+$EndComp
+Wire Wire Line
+	7050 2350 6700 2350
+Wire Wire Line
+	8300 2250 7850 2250
+Wire Wire Line
+	8300 2450 7850 2450
+Wire Wire Line
+	5900 2200 5900 3000
+Wire Wire Line
+	4400 3200 5400 3200
+Wire Wire Line
+	6900 3800 6900 4000
+Wire Wire Line
+	6900 4500 6900 4800
+Wire Wire Line
+	5100 3200 5100 3400
+Connection ~ 5100 3200
+Wire Wire Line
+	5100 3800 5100 4000
+Wire Wire Line
+	5100 4500 5100 4600
+Connection ~ 6900 4600
+Wire Wire Line
+	5900 1700 5900 1500
+Wire Wire Line
+	4400 2800 4700 2800
+Wire Wire Line
+	5900 3000 4400 3000
+Wire Wire Line
+	5200 2800 5900 2800
+Connection ~ 5900 2800
+$Comp
+L R R?
+U 1 1 52F163D6
+P 2750 3150
+F 0 "R?" V 2830 3150 40  0000 C CNN
+F 1 "R" V 2757 3151 40  0000 C CNN
+F 2 "" V 2680 3150 30  0000 C CNN
+F 3 "" H 2750 3150 30  0000 C CNN
+	1    2750 3150
+	0    1    1    0
+$EndComp
+Wire Wire Line
+	3300 3150 3000 3150
+Wire Wire Line
+	3300 2800 2000 2800
+Wire Wire Line
+	2000 3150 2500 3150
+Wire Wire Line
+	6900 3400 6900 2650
+Wire Wire Line
+	5900 2550 7050 2550
+Connection ~ 5900 2550
+Wire Wire Line
+	6700 2350 6700 1850
+Wire Wire Line
+	6700 1850 8300 1850
+Wire Wire Line
+	6900 2650 7050 2650
+Wire Wire Line
+	5100 4600 6900 4600
+$Comp
+L DIODE D?
+U 1 1 52F164E1
+P 6400 2850
+F 0 "D?" H 6400 2950 40  0000 C CNN
+F 1 "DIODE" H 6400 2750 40  0000 C CNN
+F 2 "" H 6400 2850 60  0000 C CNN
+F 3 "" H 6400 2850 60  0000 C CNN
+	1    6400 2850
+	0    -1   -1   0
+$EndComp
+Wire Wire Line
+	6400 2650 6400 2550
+Connection ~ 6400 2550
+Wire Wire Line
+	6900 3100 6400 3100
+Wire Wire Line
+	6400 3100 6400 3050
+Connection ~ 6900 3100
+Wire Wire Line
+	6600 3600 6100 3600
+Wire Wire Line
+	6100 3600 6100 3200
+Wire Wire Line
+	6100 3200 5900 3200
 $EndSCHEMATC
